File: keeb/keeb.kicad_sch (KiCad schematic)
At the start: 0 parts

Commit message: designed + inital schematic
Parts:
- added A1: RaspberryPi_Pico, Module:RaspberryPi_Pico_Common_THT, symbol MCU_Module:RaspberryPi_Pico
- added D1, D10, D11, D12, D13, D14, D15, D16, D17, D18, D19, D2, D20, D21, D22, D23, D24, D25, D26, D27, D28, D29, D3, D30, D31, D32, D33, D34, D35, D36, D37, D38, D39, D4, D40, D41, D42, D43, D44, D45, D46, D47, D48, D49, D5, D50, D51, D52, D53, D54, D55, D56, D57, D58, D59, D6, D60, D7, D8, D9: 1N4148, Diode_THT:D_DO-35_SOD27_P7.62mm_Horizontal, symbol Diode:1N4148
- added S1: MX_stab, PCM_marbastlib-mx:STAB_MX_6.25u, symbol PCM_marbastlib-mx:MX_stab
- added S2: MX_stab, PCM_marbastlib-mx:STAB_MX_2u, symbol PCM_marbastlib-mx:MX_stab
- added S3, S4: MX_stab, PCM_marbastlib-mx:STAB_MX_2.25u, symbol PCM_marbastlib-mx:MX_stab
- added S5: MX_stab, PCM_marbastlib-mx:STAB_MX_2.75u, symbol PCM_marbastlib-mx:MX_stab
- added SW1, SW10, SW11, SW12, SW13, SW14, SW15, SW16, SW17, SW18, SW19, SW2, SW20, SW21, SW22, SW23, SW24, SW25, SW26, SW27, SW28, SW29, SW3, SW30, SW31, SW32, SW33, SW34, SW35, SW36, SW37, SW38, SW39, SW4, SW40, SW41, SW42, SW43, SW44, SW45, SW46, SW47, SW48, SW49, SW5, SW50, SW51, SW52, SW53, SW54, SW55, SW56, SW57, SW58, SW59, SW6, SW60, SW7, SW8, SW9: SW_Push, PCM_marbastlib-mx:SW_MX_1u, symbol Switch:SW_Push
- added SW61: RotaryEncoder_Switch, PCM_marbastlib-various:ROT_Alps_EC11E-Switch, symbol Device:RotaryEncoder_Switch
Connections:
- new net: D7.2 (A), SW7.2
- new net: D37.2 (A), SW37.2
- new net: D6.2 (A), SW6.2
- new net: D43.2 (A), SW43.2
- new net: D53.2 (A), SW53.2
- new net: D34.2 (A), SW34.2
- new net: D24.2 (A), SW24.2
- new net: D22.2 (A), SW22.2
- new net: D52.2 (A), SW52.2
- new net: D11.2 (A), SW11.2
- new net: D5.2 (A), SW5.2
- new net: D42.2 (A), SW42.2
- new net: D17.2 (A), SW17.2
- new net: D8.2 (A), SW8.2
- new net: D54.2 (A), SW54.2
- new net: D26.2 (A), SW26.2
- new net: D1.2 (A), SW1.2
- new net: D50.2 (A), SW50.2
- new net: D48.2 (A), SW48.2
- new net: D14.2 (A), SW14.2
- new net: D58.2 (A), SW58.2
- new net: D12.2 (A), SW12.2
- new net: D49.2 (A), SW49.2
- new net: D32.2 (A), SW32.2
- new net: D46.2 (A), SW46.2
- new net: D60.2 (A), SW60.2
- new net: D27.2 (A), SW27.2
- new net: D30.2 (A), SW30.2
- new net: D40.2 (A), SW40.2
- new net: D56.2 (A), SW56.2
- new net: D38.2 (A), SW38.2
- new net: D45.2 (A), SW45.2
- new net: D28.2 (A), SW28.2
- new net: D39.2 (A), SW39.2
- new net: D15.2 (A), SW15.2
- new net: D25.2 (A), SW25.2
- new net: D3.2 (A), SW3.2
- new net: D18.2 (A), SW18.2
- new net: D51.2 (A), SW51.2
- new net: D35.2 (A), SW35.2
- new net: D59.2 (A), SW59.2
- new net: D19.2 (A), SW19.2
- new net: D23.2 (A), SW23.2
- new net: D16.2 (A), SW16.2
- new net: D55.2 (A), SW55.2
- new net: D20.2 (A), SW20.2
- new net: D2.2 (A), SW2.2
- new net: D57.2 (A), SW57.2
- new net: D10.2 (A), SW10.2
- new net: D13.2 (A), SW13.2
- new net: D21.2 (A), SW21.2
- new net: D47.2 (A), SW47.2
- new net: D29.2 (A), SW29.2
- new net: D44.2 (A), SW44.2
- new net: D36.2 (A), SW36.2
- new net: D4.2 (A), SW4.2
- new net: D9.2 (A), SW9.2
- new net: D31.2 (A), SW31.2
- new net: D41.2 (A), SW41.2
- new net: D33.2 (A), SW33.2
- new net COL0: A1.7 (GPIO5), SW1.1, SW2.1, SW3.1, SW4.1, SW5.1
- new net COL1: A1.9 (GPIO6), SW10.1, SW6.1, SW7.1, SW8.1, SW9.1
- new net COL10: A1.19 (GPIO14), SW48.1, SW49.1, SW50.1, SW51.1
- new net COL11: A1.20 (GPIO15), SW52.1, SW53.1, SW54.1, SW55.1
- new net COL12: A1.21 (GPIO16), SW56.1, SW57.1, SW58.1
- new net COL13: A1.22 (GPIO17), SW59.1, SW60.1, SW61.S1
- new net COL2: SW11.1, SW12.1, SW13.1, SW14.1, SW15.1
- new net COL3: A1.10 (GPIO7), SW16.1, SW17.1, SW18.1, SW19.1, SW20.1
- new net COL4: A1.11 (GPIO8), SW21.1, SW22.1, SW23.1, SW24.1, SW25.1
- new net COL5: A1.12 (GPIO9), SW26.1, SW27.1, SW28.1, SW29.1, SW30.1
- new net COL6: A1.14 (GPIO10), SW31.1, SW32.1, SW33.1, SW34.1, SW35.1
- new net COL7: A1.15 (GPIO11), SW36.1, SW37.1, SW38.1, SW39.1
- new net COL8: A1.16 (GPIO12), SW40.1, SW41.1, SW42.1, SW43.1
- new net COL9: A1.17 (GPIO13), SW44.1, SW45.1, SW46.1, SW47.1
- new net GND: A1.13 (GND), A1.18 (GND), A1.23 (GND), A1.28 (GND), A1.3 (GND), A1.38 (GND), A1.8 (GND), SW61.C
- new net RE0: A1.24 (GPIO18), SW61.A
- new net RE1: A1.25 (GPIO19), SW61.B
- new net ROW0: A1.1 (GPIO0), D1.1 (K), D11.1 (K), D16.1 (K), D21.1 (K), D26.1 (K), D31.1 (K), D36.1 (K), D40.1 (K), D44.1 (K), D48.1 (K), D52.1 (K), D56.1 (K), D59.1 (K), D6.1 (K)
- new net ROW1: A1.2 (GPIO1), D12.1 (K), D17.1 (K), D2.1 (K), D22.1 (K), D27.1 (K), D32.1 (K), D37.1 (K), D41.1 (K), D45.1 (K), D49.1 (K), D53.1 (K), D57.1 (K), D60.1 (K), D7.1 (K)
- new net ROW2: A1.4 (GPIO2), D13.1 (K), D18.1 (K), D23.1 (K), D28.1 (K), D3.1 (K), D33.1 (K), D38.1 (K), D42.1 (K), D46.1 (K), D50.1 (K), D54.1 (K), D58.1 (K), D8.1 (K), SW61.S2
- new net ROW3: A1.5 (GPIO3), D14.1 (K), D19.1 (K), D24.1 (K), D29.1 (K), D34.1 (K), D39.1 (K), D4.1 (K), D43.1 (K), D47.1 (K), D51.1 (K), D55.1 (K), D9.1 (K)
- new net ROW4: A1.6 (GPIO4), D10.1 (K), D15.1 (K), D20.1 (K), D25.1 (K), D30.1 (K), D35.1 (K), D5.1 (K)
- no-connect marks 0 -> 13

Commit message: made v1 of pcb design + traced v1
Parts:
- added D61: 1N4148, Diode_THT:D_DO-35_SOD27_P7.62mm_Horizontal, symbol Diode:1N4148
Connections:
- net COL10: now also A1.20 (GPIO15); no longer A1.19 (GPIO14)
- net COL11: now also A1.21 (GPIO16); no longer A1.20 (GPIO15)
- net COL12: now also A1.22 (GPIO17); no longer A1.21 (GPIO16)
- net COL13: now also A1.24 (GPIO18); no longer A1.22 (GPIO17)
- net COL2: now also A1.10 (GPIO7)
- net COL3: now also A1.11 (GPIO8); no longer A1.10 (GPIO7)
- net COL4: now also A1.12 (GPIO9); no longer A1.11 (GPIO8)
- net COL5: now also A1.14 (GPIO10); no longer A1.12 (GPIO9)
- net COL6: now also A1.15 (GPIO11); no longer A1.14 (GPIO10)
- net COL7: now also A1.16 (GPIO12); no longer A1.15 (GPIO11)
- net COL8: now also A1.17 (GPIO13); no longer A1.16 (GPIO12)
- net COL9: now also A1.19 (GPIO14); no longer A1.17 (GPIO13)
- net RE0: now also A1.25 (GPIO19); no longer A1.24 (GPIO18)
- net RE1: now also A1.26 (GPIO20); no longer A1.25 (GPIO19)
- net ROW2: now also D61.1 (K); no longer SW61.S2
- new net: D61.2 (A), SW61.S2
- no-connect marks 13 -> 12
Changed lines of the file:
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@@
 	)
 	(no_connect
-		(at 271.78 124.46)
-	)
-	(no_connect
 		(at 248.92 88.9)
 	)
@@
 	(wire
 		(pts
-			(xy 271.78 119.38) (xy 274.32 119.38)
+			(xy 176.53 48.26) (xy 189.23 48.26)
 		)
 		(stroke
@@
 	(wire
 		(pts
-			(xy 176.53 48.26) (xy 189.23 48.26)
+			(xy 220.98 134.62) (xy 226.06 134.62)
 		)
 		(stroke
@@
 	(wire
 		(pts
-			(xy 220.98 134.62) (xy 226.06 134.62)
+			(xy 114.3 86.36) (xy 127 86.36)
 		)
 		(stroke
@@
 	(wire
 		(pts
-			(xy 114.3 86.36) (xy 127 86.36)
+			(xy 191.77 29.21) (xy 191.77 39.37)
 		)
 		(stroke
@@
 	(wire
 		(pts
-			(xy 191.77 29.21) (xy 191.77 39.37)
+			(xy 204.47 59.69) (xy 204.47 71.12)
 		)
 		(stroke
@@
 	(wire
 		(pts
-			(xy 204.47 59.69) (xy 204.47 71.12)
+			(xy 271.78 121.92) (xy 274.32 121.92)
 		)
 		(stroke
@@
 	(wire
 		(pts
+			(xy 238.76 85.09) (xy 238.76 88.9)
+		)
+		(stroke
+			(width 0)
+			(type default)
+		)
+	)
+	(wire
+		(pts
 			(xy 115.57 29.21) (xy 115.57 39.37)
 		)
@@
 	(wire
 		(pts
+			(xy 238.76 88.9) (xy 204.47 88.9)
+		)
+		(stroke
+			(width 0)
+			(type default)
+		)
+	)
+	(wire
+		(pts
 			(xy 201.93 39.37) (xy 201.93 40.64)
 		)
@@
 	(wire
 		(pts
-			(xy 204.47 88.9) (xy 231.14 88.9)
+			(xy 62.23 77.47) (xy 62.23 78.74)
 		)
 		(stroke
@@
 	(wire
 		(pts
-			(xy 62.23 77.47) (xy 62.23 78.74)
+			(xy 127 86.36) (xy 139.7 86.36)
 		)
 		(stroke
@@
 	(wire
 		(pts
-			(xy 127 86.36) (xy 139.7 86.36)
+			(xy 101.6 77.47) (xy 101.6 78.74)
 		)
 		(stroke
@@
 	(wire
 		(pts
-			(xy 101.6 77.47) (xy 101.6 78.74)
+			(xy 116.84 77.47) (xy 116.84 95.25)
 		)
 		(stroke
@@
 	(wire
 		(pts
-			(xy 116.84 77.47) (xy 116.84 95.25)
+			(xy 271.78 116.84) (xy 274.32 116.84)
 		)
 		(stroke
@@
 	(wire
 		(pts
+			(xy 271.78 119.38) (xy 274.32 119.38)
+		)
+		(stroke
+			(width 0)
+			(type default)
+		)
+	)
+	(wire
+		(pts
 			(xy 60.96 39.37) (xy 60.96 40.64)
 		)
@@
 	(wire
 		(pts
+			(xy 271.78 124.46) (xy 276.86 124.46)
+		)
+		(stroke
+			(width 0)
+			(type default)
+		)
+	)
+	(wire
+		(pts
 			(xy 204.47 29.21) (xy 204.47 39.37)
 		)
@@
 	(wire
 		(pts
-			(xy 231.14 88.9) (xy 231.14 85.09)
-		)
-		(stroke
-			(width 0)
-			(type default)
-		)
-	)
-	(wire
-		(pts
 			(xy 166.37 29.21) (xy 166.37 39.37)
 		)
@@
 	(wire
 		(pts
-			(xy 101.6 86.36) (xy 114.3 86.36)
+			(xy 271.78 114.3) (xy 274.32 114.3)
 		)
 		(stroke
@@
 	(wire
 		(pts
-			(xy 165.1 68.58) (xy 177.8 68.58)
+			(xy 101.6 86.36) (xy 114.3 86.36)
 		)
 		(stroke
@@
 	(wire
 		(pts
-			(xy 52.07 95.25) (xy 52.07 114.3)
+			(xy 165.1 68.58) (xy 177.8 68.58)
 		)
 		(stroke
@@
 	(wire
 		(pts
-			(xy 163.83 39.37) (xy 163.83 40.64)
+			(xy 52.07 95.25) (xy 52.07 114.3)
 		)
 		(stroke
@@
 	(wire
 		(pts
-			(xy 46.99 39.37) (xy 46.99 40.64)
+			(xy 163.83 39.37) (xy 163.83 40.64)
 		)
 		(stroke
@@
 	(wire
 		(pts
-			(xy 128.27 39.37) (xy 128.27 59.69)
+			(xy 46.99 39.37) (xy 46.99 40.64)
 		)
 		(stroke
@@
 	(wire
 		(pts
-			(xy 128.27 29.21) (xy 128.27 39.37)
+			(xy 128.27 39.37) (xy 128.27 59.69)
 		)
 		(stroke
@@
 	(wire
 		(pts
-			(xy 204.47 39.37) (xy 204.47 59.69)
+			(xy 128.27 29.21) (xy 128.27 39.37)
 		)
 		(stroke
@@
 	(wire
 		(pts
-			(xy 271.78 116.84) (xy 274.32 116.84)
+			(xy 204.47 39.37) (xy 204.47 59.69)
 		)
 		(stroke
@@
 	(wire
 		(pts
-			(xy 271.78 121.92) (xy 276.86 121.92)
-		)
-		(stroke
-			(width 0)
-			(type default)
-		)
-	)
-	(wire
-		(pts
 			(xy 104.14 59.69) (xy 104.14 57.15)
 		)
@@
 	(wire
 		(pts
-			(xy 271.78 114.3) (xy 274.32 114.3)
-		)
-		(stroke
-			(width 0)
-			(type default)
-		)
-	)
-	(wire
-		(pts
 			(xy 125.73 48.26) (xy 138.43 48.26)
 		)
@@
 		)
 	)
-	(label "COL6"
+	(label "COL5"
 		(at 220.98 137.16 0)
 		(effects
@@
 		)
 	)
-	(label "COL7"
+	(label "COL6"
 		(at 220.98 139.7 0)
 		(effects
@@
 		)
 	)
-	(label "COL10"
+	(label "COL9"
 		(at 220.98 147.32 0)
 		(effects
@@
 	)
 	(label "RE1"
-		(at 276.86 121.92 0)
+		(at 276.86 124.46 0)
 		(effects
 			(font
@@
 		)
 	)
-	(label "COL5"
+	(label "COL4"
 		(at 220.98 134.62 0)
 		(effects
@@
 		)
 	)
-	(label "COL9"
+	(label "COL8"
 		(at 220.98 144.78 0)
 		(effects
@@
 	)
 	(label "COL12"
-		(at 274.32 114.3 0)
+		(at 274.32 116.84 0)
 		(effects
 			(font
@@
 		)
 	)
-	(label "COL8"
+	(label "COL7"
 		(at 220.98 142.24 0)
 		(effects
@@
 		)
 	)
-	(label "COL3"
+	(label "COL2"
 		(at 220.98 129.54 0)
 		(effects
@@
 	)
 	(label "COL13"
-		(at 274.32 116.84 0)
+		(at 274.32 119.38 0)
 		(effects
 			(font
@@
 	)
 	(label "RE0"
-		(at 274.32 119.38 0)
+		(at 274.32 121.92 0)
 		(effects
 			(font
@@
 		)
 	)
-	(label "COL11"
+	(label "COL10"
 		(at 219.71 149.86 0)
 		(effects
@@
 		)
 	)
-	(label "COL4"
+	(label "COL3"
 		(at 220.98 132.08 0)
 		(effects
@@
 		)
 	)
+	(label "COL11"
+		(at 274.32 114.3 0)
+		(effects
+			(font
+				(size 1.27 1.27)
+			)
+			(justify left bottom)
+		)
+	)
 	(label "ROW2"
 		(at 25.4 85.09 0)
@@
 					(unit 1)
 				)
+			)
+		)
+	)
+	(symbol
+		(lib_id "Diode:1N4148")
+		(at 234.95 85.09 180)
+		(unit 1)
+		(body_style 1)
+		(exclude_from_sim no)
+		(in_bom yes)
+		(on_board yes)
+		(in_pos_files yes)
+		(dnp no)
+		(fields_autoplaced yes)
+		(property "Reference" "D61"
+			(at 234.95 78.74 0)
+			(show_name no)
+			(do_not_autoplace no)
+			(effects
+				(font
+					(size 1.27 1.27)
+				)
+			)
+		)
+		(property "Value" "1N4148"
+			(at 234.95 81.28 0)
+			(show_name no)
+			(do_not_autoplace no)
+			(effects
+				(font
+					(size 1.27 1.27)
+				)
+			)
+		)
+		(property "Footprint" "Diode_THT:D_DO-35_SOD27_P7.62mm_Horizontal"
+			(at 234.95 85.09 0)
+			(hide yes)
+			(show_name no)
+			(do_not_autoplace no)
+			(effects
+				(font
+					(size 1.27 1.27)
+				)
+			)
+		)
+		(property "Datasheet" "https://assets.nexperia.com/documents/data-sheet/1N4148_1N4448.pdf"
+			(at 234.95 85.09 0)
+			(hide yes)
+			(show_name no)
+			(do_not_autoplace no)
+			(effects
+				(font
+					(size 1.27 1.27)
+				)
+			)
+		)
+		(property "Description" "100V 0.15A standard switching diode, DO-35"
+			(at 234.95 85.09 0)
+			(hide yes)
+			(show_name no)
+			(do_not_autoplace no)
+			(effects
+				(font
+					(size 1.27 1.27)
+				)
+			)
+		)
+		(property "Sim.Device" "D"
+			(at 234.95 85.09 0)
+			(hide yes)
+			(show_name no)
+			(do_not_autoplace no)
+			(effects
+				(font
+					(size 1.27 1.27)
+				)
+			)
+		)
+		(property "Sim.Pins" "1=K 2=A"
+			(at 234.95 85.09 0)
+			(hide yes)
+			(show_name no)
+			(do_not_autoplace no)
+			(effects
+				(font
+					(size 1.27 1.27)
+				)
+			)
+		)
+		(pin "2"
+		)
+		(pin "1"
+		)
+		(instances
+			(project "keeb"
+				(path "/b87323b3-a491-4636-afec-3f7bdb012fbf"
+					(reference "D61")
+					(unit 1)
+				)
