File: keeb/keeb.kicad_pcb (KiCad board)
At the start: 2 copper layers, 337.3 x 104 mm, 128 parts, among them SW1 SW_Push, SW10 SW_Push, SW11 SW_Push, SW12 SW_Push, SW13 SW_Push, SW14 SW_Push, SW15 SW_Push, SW16 SW_Push, SW17 SW_Push, SW18 SW_Push, SW19 SW_Push, SW2 SW_Push, SW20 SW_Push, SW21 SW_Push, SW22 SW_Push, SW23 SW_Push, SW24 SW_Push, SW25 SW_Push, SW26 SW_Push, SW27 SW_Push, SW28 SW_Push, SW29 SW_Push, SW3 SW_Push, SW30 SW_Push, SW31 SW_Push, SW32 SW_Push, SW33 SW_Push, SW34 SW_Push, SW35 SW_Push, SW36 SW_Push, SW37 SW_Push, SW38 SW_Push, SW39 SW_Push, SW4 SW_Push, SW40 SW_Push, SW41 SW_Push, SW42 SW_Push, SW43 SW_Push, SW44 SW_Push, SW45 SW_Push, SW46 SW_Push, SW47 SW_Push, SW48 SW_Push, SW49 SW_Push, SW5 SW_Push, SW50 SW_Push, SW51 SW_Push, SW52 SW_Push, SW53 SW_Push, SW54 SW_Push, SW55 SW_Push, SW56 SW_Push, SW57 SW_Push, SW58 SW_Push, SW59 SW_Push, SW6 SW_Push, SW60 SW_Push, SW61 RotaryEncoder_Switch, SW7 SW_Push, SW8 SW_Push, SW9 SW_Push

Commit message: entry 3, pcb files final + custom silk screen art
Parts:
- added G***: LOGO, custom:art, F.Cu at (160.3, 59.9)
- moved D61 15.2 mm to (7.14, 41.1)
Routing:
- net /GND: track 546.4 -> 853.8 mm, vias 0 -> 4
- net /RE0: track 419.2 -> 433.8 mm
- net Net-(D61-A): track 12.7 -> 21.2 mm
- net Net-(D41-A): track 0.00 -> 8.50 mm
- net /RE1: track 376.4 -> 383.9 mm
- net /ROW2: track 366.8 -> 361.5 mm
- added copper zone on B.Cu, net /GND
- added copper zone on F.Cu, net /GND
